Commit message: seperate robot description file from simulation package

File: src/usv_description/urdf/usv.urdf (robot description, URDF)
Before this commit: robot blueboat_usv, 1 links, 0 joints
Links:
- added link imu_link
- added link laser_link
- added link left_prop
- added link left_wing; collision box size=0.2 0.05 0.05; visual box size=0.2 0.05 0.05
- added link right_prop
- added link right_wing; collision box size=0.2 0.05 0.05; visual box size=0.2 0.05 0.05
- link base_link: geometry collision capsule length=0.5 radius=0.1; visual capsule length=0.5 radius=0.1
Joints:
- added joint imu_joint: type fixed, parent base_link, child imu_link, origin xyz=0 0 0 rpy=0 0 0
- added joint laser_joint: type fixed, parent base_link, child laser_link, origin xyz=0 -0.15 0 rpy=3.14159 0 1.5708
- added joint left_prop_joint: type continuous, parent base_link, child left_prop, origin xyz=-0.25 0 0.005 rpy=0 3.14159 0, axis 0 0 -1
- added joint left_wing_joint: type fixed, parent base_link, child left_wing, origin xyz=-0.15 0 0.05 rpy=0 0 0
- added joint right_prop_joint: type continuous, parent base_link, child right_prop, origin xyz=0.25 0 0.005 rpy=0 3.14159 0, axis 0 0 -1
- added joint right_wing_joint: type fixed, parent base_link, child right_wing, origin xyz=0.15 0 0.05 rpy=0 0 0

Commit message: feat: redo urdf/wbt files to have sane axis alignments, tuned Nav2 parameters to pass the same path test as pre-refactor, add custom "backup" behavior tree,

File: src/usv_description/urdf/usv.urdf (robot description, URDF)
Before this commit: robot my_robot, 7 links, 6 joints
Joints:
- joint laser_joint: origin xyz=0 -0.15 0 rpy=3.14159 0 1.5708 -> xyz=0.2 0 0.2 rpy=0 0 0
- joint left_prop_joint: axis 0 0 -1 -> 1 0 0; origin xyz=-0.25 0 0.005 rpy=0 3.14159 0 -> xyz=-0.25 0.1 0.005 rpy=0 0 0
- joint left_wing_joint: origin xyz=-0.15 0 0.05 rpy=0 0 0 -> xyz=0 0.15 0.05 rpy=0 0 0
- joint right_prop_joint: axis 0 0 -1 -> 1 0 0; origin xyz=0.25 0 0.005 rpy=0 3.14159 0 -> xyz=-0.25 -0.1 0.005 rpy=0 0 0
- joint right_wing_joint: origin xyz=0.15 0 0.05 rpy=0 0 0 -> xyz=0 -0.15 0.05 rpy=0 0 0

Commit message: change to using blueboat cad model (excluding large STL)

File: src/usv_description/urdf/usv.urdf (robot description, URDF)
Before this commit: robot my_robot, 7 links, 6 joints
Links:
- removed link left_wing
- removed link right_wing
- link base_link: geometry collision box size=1.2 0.75 0.4; visual mesh filename=package://usv_description/meshes/blueboat_visual.obj
Joints:
- removed joint left_wing_joint
- removed joint right_wing_joint
- joint laser_joint: origin xyz=0.2 0 0.2 rpy=0 0 0 -> xyz=0 0 0.0 rpy=0 0 0
- joint left_prop_joint: origin xyz=-0.25 0.1 0.005 rpy=0 0 0 -> xyz=-0.45 0.25 0.005 rpy=0 0 0
- joint right_prop_joint: origin xyz=-0.25 -0.1 0.005 rpy=0 0 0 -> xyz=-0.45 -0.25 0.005 rpy=0 0 0
